Commit message: Chassis joint coordinates correct

File: src/robotics_configurations/alex_description/robots/alex.urdf.xacro (robot description, xacro)
@@ -2,5 +2,5 @@
 <robot xmlns:xacro="http://www.ros.org/wiki/xacro" name="alex">
     <material name="grey">
-        <color rgba="0.75 0.75 0.75 1"/>
+        <color rgba="0.75 0.75 0.75 0.5"/>
     </material>
     <material name="red">
@@ -22,11 +22,24 @@
         </visual>
     </link>
-    <xacro:property name="chassis_mass" value="0.05"/>
-    <xacro:property name="chassis_length" value="0.276"/>
-    <xacro:property name="chassis_width" value="0.192"/>
-    <xacro:property name="chassis_height" value="0.059"/>
-    <xacro:property name="chassis_ixx" value="${(chassis_mass / 12.0) * (chassis_length**2 + chassis_height**2)}"/>
-    <xacro:property name="chassis_iyy" value="${(chassis_mass / 12.0) * (chassis_width**2 + chassis_height**2)}"/>
-    <xacro:property name="chassis_izz" value="${(chassis_mass / 12.0) * (chassis_width**2 + chassis_length**2)}"/>
+    <!-- Chassis Properties -->
+    <xacro:property name="chassis_mass" value="0.1"/>
+    <xacro:property name="chassis_width_x" value="0.192"/>
+    <xacro:property name="chassis_depth_y" value="0.059"/>
+    <xacro:property name="chassis_height_z" value="0.276"/>
+    <xacro:property name="chassis_ixx" value="${(chassis_mass / 12.0) * (chassis_depth_y**2 + chassis_height_z**2)}"/>
+    <xacro:property name="chassis_iyy" value="${(chassis_mass / 12.0) * (chassis_width_x**2 + chassis_height_z**2)}"/>
+    <xacro:property name="chassis_izz" value="${(chassis_mass / 12.0) * (chassis_width_x**2 + chassis_depth_y**2)}"/>
+    <xacro:macro name="chassis_joint_origin">
+        <origin xyz="-0.068 0 0.056475" rpy="${pi/2} 0 ${-pi/2}"/>
+    </xacro:macro>
+    <!-- * * * * * * * * * -->
+    <!-- Wheel Properties -->
+    <xacro:property name="wheel_mass" value="0.01"/>
+    <xacro:property name="wheel_width" value="0.029"/>
+    <xacro:property name="wheel_radius" value="0.0375"/>
+    <xacro:property name="wheel_ixx" value="${(wheel_mass / 12.0) * (3 * wheel_radius**2 + wheel_width**2)}"/>
+    <xacro:property name="wheel_iyy" value="${wheel_ixx}"/>
+    <xacro:property name="wheel_izz" value="${(chassis_mass * wheel_radius**2) / 2}"/>
+    <!-- * * * * * * * * * -->
     <link name="chassis">
         <inertial>
@@ -38,5 +51,5 @@
             <origin rpy="0 0 0" xyz="0 0 0"/>
             <geometry>
-                <box size="${chassis_length} ${chassis_width} ${chassis_height}"/>
+                <box size="${chassis_width_x} ${chassis_depth_y} ${chassis_height_z}"/>
             </geometry>
             <material name="grey"/>
@@ -45,5 +58,5 @@
             <origin rpy="0 0 0" xyz="0 0 0"/>
             <geometry>
-                <box size="${chassis_length} ${chassis_width} ${chassis_height}"/>
+                <box size="${chassis_width_x} ${chassis_depth_y} ${chassis_height_z}"/>
             </geometry>
         </collision>
@@ -52,5 +65,5 @@
     	<parent link="base_link"/>
     	<child link="chassis"/>
-    	<origin xyz="0 0 0" rpy="0 0 0"/>
+    	<xacro:chassis_joint_origin/>
 	</joint>
     <!--<link name="castor_swivel">

Commit message: Add wheel cylinder link/joint and fix chassis origin

File: src/robotics_configurations/alex_description/robots/alex.urdf.xacro (robot description, xacro)
@@ -13,13 +13,4 @@
         <color rgba="0 0.7 0.64 1"/>
     </material>
-    <link name="base_link">
-        <visual>
-            <origin rpy="0.0 0 0" xyz="0 0 0"/>
-            <geometry>
-                <box size="0.01 0.01 0.01"/>
-            </geometry>
-            <material name="red"/>
-        </visual>
-    </link>
     <!-- Chassis Properties -->
     <xacro:property name="chassis_mass" value="0.1"/>
@@ -30,4 +21,7 @@
     <xacro:property name="chassis_iyy" value="${(chassis_mass / 12.0) * (chassis_width_x**2 + chassis_height_z**2)}"/>
     <xacro:property name="chassis_izz" value="${(chassis_mass / 12.0) * (chassis_width_x**2 + chassis_depth_y**2)}"/>
+    <xacro:macro name="chassis_origin">
+        <origin xyz="0 ${-chassis_depth_y/2} 0" rpy="0 0 0"/>
+    </xacro:macro>
     <xacro:macro name="chassis_joint_origin">
         <origin xyz="-0.068 0 0.056475" rpy="${pi/2} 0 ${-pi/2}"/>
@@ -41,13 +35,37 @@
     <xacro:property name="wheel_iyy" value="${wheel_ixx}"/>
     <xacro:property name="wheel_izz" value="${(chassis_mass * wheel_radius**2) / 2}"/>
+    <xacro:macro name="right_wheel_joint_origin">
+        <origin xyz="0 -0.0805 0" rpy="${-pi/2} 0 0"/>
+    </xacro:macro>
     <!-- * * * * * * * * * -->
+    <!-- Macros -->
+    <xacro:macro name="x_axis">
+        <axis xyz="1 0 0"/>
+    </xacro:macro>
+    <xacro:macro name="y_axis">
+        <axis xyz="0 1 0"/>
+    </xacro:macro>
+    <xacro:macro name="z_axis">
+        <axis xyz="0 0 1"/>
+    </xacro:macro>
+    <!-- * * * * * * * * * -->
+    <!-- Model Definitions -->
+    <link name="base_link">
+        <visual>
+            <origin rpy="0.0 0 0" xyz="0 0 0"/>
+            <geometry>
+                <box size="0.01 0.01 0.01"/>
+            </geometry>
+            <material name="red"/>
+        </visual>
+    </link>
     <link name="chassis">
         <inertial>
-            <origin rpy="0 0 0" xyz="0 0 0"/>
+            <xacro:chassis_origin/>
             <mass value="${chassis_mass}"/>
             <inertia ixx="${chassis_ixx}" ixy="0.0" ixz="0.0" iyy="${chassis_iyy}" iyz="0.0" izz="${chassis_izz}"/>
         </inertial>
         <visual>
-            <origin rpy="0 0 0" xyz="0 0 0"/>
+            <xacro:chassis_origin/>
             <geometry>
                 <box size="${chassis_width_x} ${chassis_depth_y} ${chassis_height_z}"/>
@@ -56,5 +74,5 @@
         </visual>
         <collision>
-            <origin rpy="0 0 0" xyz="0 0 0"/>
+            <xacro:chassis_origin/>
             <geometry>
                 <box size="${chassis_width_x} ${chassis_depth_y} ${chassis_height_z}"/>
@@ -62,8 +80,35 @@
         </collision>
     </link>
-    <joint name="fixed" type="fixed">
+    <joint name="baselink_chassis_joint" type="fixed">
     	<parent link="base_link"/>
     	<child link="chassis"/>
     	<xacro:chassis_joint_origin/>
+	</joint>
+    <link name="right_wheel">
+        <inertial>
+            <origin rpy="0 0 0" xyz="0 0 0"/>
+            <mass value="${wheel_mass}"/>
+            <inertia ixx="${wheel_ixx}" ixy="0.0" ixz="0.0" iyy="${wheel_iyy}" iyz="0.0" izz="${wheel_izz}"/>
+        </inertial>
+        <visual>
+            <origin rpy="0 0 0" xyz="0 0 0"/>
+            <geometry>
+                <cylinder radius="${wheel_radius}" length="${wheel_width}"/>
+            </geometry>
+            <material name="black"/>
+        </visual>
+        <collision>
+            <origin rpy="0 0 0" xyz="0 0 0"/>
+            <geometry>
+                <cylinder radius="${wheel_radius}" length="${wheel_width}"/>
+            </geometry>
+        </collision>
+    </link>
+    <joint name="baselink_right_wheel_joint" type="continuous">
+    	<parent link="base_link"/>
+    	<child link="right_wheel"/>
+    	<xacro:right_wheel_joint_origin/>
+        <limit effort="1.0" velocity="0.005"/>
+        <xacro:z_axis/>
 	</joint>
     <!--<link name="castor_swivel">

Commit message: Add joint controller GUI and fix missing TF transform for wheel

File: src/robotics_configurations/alex_description/robots/alex.urdf.xacro (robot description, xacro)
@@ -109,5 +109,5 @@
     	<child link="right_wheel"/>
     	<xacro:right_wheel_joint_origin/>
-        <limit effort="1.0" velocity="0.005"/>
+        <limit effort="1.0" velocity="0.45"/>
         <xacro:z_axis/>
 	</joint>

Commit message: Add second wheel

File: src/robotics_configurations/alex_description/robots/alex.urdf.xacro (robot description, xacro)
@@ -38,4 +38,7 @@
         <origin xyz="0 -0.0805 0" rpy="${-pi/2} 0 0"/>
     </xacro:macro>
+    <xacro:macro name="left_wheel_joint_origin">
+        <origin xyz="0 0.0805 0" rpy="${pi/2} 0 0"/>
+    </xacro:macro>
     <!-- * * * * * * * * * -->
     <!-- Macros -->
@@ -52,4 +55,5 @@
     <!-- Model Definitions -->
     <link name="base_link">
+        <pose>0 0 ${wheel_radius} 0 0 0</pose>
         <visual>
             <origin rpy="0.0 0 0" xyz="0 0 0"/>
@@ -112,4 +116,31 @@
         <xacro:z_axis/>
 	</joint>
+    <link name="left_wheel">
+        <inertial>
+            <origin rpy="0 0 0" xyz="0 0 0"/>
+            <mass value="${wheel_mass}"/>
+            <inertia ixx="${wheel_ixx}" ixy="0.0" ixz="0.0" iyy="${wheel_iyy}" iyz="0.0" izz="${wheel_izz}"/>
+        </inertial>
+        <visual>
+            <origin rpy="0 0 0" xyz="0 0 0"/>
+            <geometry>
+                <cylinder radius="${wheel_radius}" length="${wheel_width}"/>
+            </geometry>
+            <material name="black"/>
+        </visual>
+        <collision>
+            <origin rpy="0 0 0" xyz="0 0 0"/>
+            <geometry>
+                <cylinder radius="${wheel_radius}" length="${wheel_width}"/>
+            </geometry>
+        </collision>
+    </link>
+    <joint name="baselink_left_wheel_joint" type="continuous">
+    	<parent link="base_link"/>
+    	<child link="left_wheel"/>
+    	<xacro:left_wheel_joint_origin/>
+        <limit effort="1.0" velocity="0.45"/>
+        <xacro:z_axis/>
+	</joint>
     <!--<link name="castor_swivel">
     </link>

Commit message: Working gazebo simulation of two-wheeled robot

File: src/robotics_configurations/alex_description/robots/alex.urdf.xacro (robot description, xacro)
@@ -13,4 +13,31 @@
         <color rgba="0 0.7 0.64 1"/>
     </material>
+    <!-- Gazebo parameters -->
+    <gazebo>
+        <plugin filename="libgazebo_ros_diff_drive.so" name="differential_drive_controller">
+            <legacyMode>false</legacyMode>
+            <alwaysOn>true</alwaysOn>
+            <updateRate>20</updateRate>
+            <leftJoint>baselink_left_wheel_joint</leftJoint>
+            <rightJoint>baselink_right_wheel_joint</rightJoint>
+            <wheelSeparation>0.0175</wheelSeparation>
+            <wheelDiameter>0.075</wheelDiameter>
+            <torque>0.01</torque>
+            <commandTopic>cmd_vel</commandTopic>
+            <odometryTopic>odom</odometryTopic>
+            <odometryFrame>odom</odometryFrame>
+            <robotBaseFrame>base_link</robotBaseFrame>
+        </plugin>
+    </gazebo>
+    <xacro:macro name="gazebo_params" params="link_ref">
+        <gazebo reference="${link_ref}">
+            <kp>100.0</kp>
+            <kd>100.0</kd>
+            <mu1>10.0</mu1>
+            <mu2>10.0</mu2>
+            <!--<xacro:insert_block name="material" />-->
+<!--            <material>Gazebo/${material}</material>-->
+        </gazebo>
+    </xacro:macro>
     <!-- Chassis Properties -->
     <xacro:property name="chassis_mass" value="0.1"/>
@@ -39,16 +66,16 @@
     </xacro:macro>
     <xacro:macro name="left_wheel_joint_origin">
-        <origin xyz="0 0.0805 0" rpy="${pi/2} 0 0"/>
+        <origin xyz="0 0.0805 0" rpy="${-pi/2} 0 0"/>
     </xacro:macro>
     <!-- * * * * * * * * * -->
     <!-- Macros -->
     <xacro:macro name="x_axis">
-        <axis xyz="1 0 0"/>
+        <axis xyz="1 0 0" rpy="0 0 0"/>
     </xacro:macro>
     <xacro:macro name="y_axis">
-        <axis xyz="0 1 0"/>
+        <axis xyz="0 1 0" rpy="0 0 0"/>
     </xacro:macro>
     <xacro:macro name="z_axis">
-        <axis xyz="0 0 1"/>
+        <axis xyz="0 0 1" rpy="0 0 0"/>
     </xacro:macro>
     <!-- * * * * * * * * * -->
@@ -115,4 +142,5 @@
         <limit effort="1.0" velocity="0.45"/>
         <xacro:z_axis/>
+        <joint_properties damping="1.0" friction="1.0"/>
 	</joint>
     <link name="left_wheel">
@@ -142,5 +170,8 @@
         <limit effort="1.0" velocity="0.45"/>
         <xacro:z_axis/>
+        <joint_properties damping="1.0" friction="1.0"/>
 	</joint>
+    <xacro:gazebo_params link_ref="left_wheel"/>
+    <xacro:gazebo_params link_ref="right_wheel"/>
     <!--<link name="castor_swivel">
     </link>

Commit message: Add castor and castor wheel, add STLs for chassis and castor wheel

File: src/robotics_configurations/alex_description/robots/alex.urdf.xacro (robot description, xacro)
@@ -2,5 +2,5 @@
 <robot xmlns:xacro="http://www.ros.org/wiki/xacro" name="alex">
     <material name="grey">
-        <color rgba="0.75 0.75 0.75 0.5"/>
+        <color rgba="0.75 0.75 0.75 1.0"/>
     </material>
     <material name="red">
@@ -8,5 +8,5 @@
     </material>
     <material name="black">
-        <color rgba="0.8 0.8 0.8 1"/>
+        <color rgba="1.0 1.0 1.0 1"/>
     </material>
     <material name="pi-top_green">
@@ -30,5 +30,5 @@
         </plugin>
     </gazebo>
-    <xacro:macro name="gazebo_params" params="link_ref">
+    <xacro:macro name="gazebo_wheel_params" params="link_ref">
         <gazebo reference="${link_ref}">
             <kp>100.0</kp>
@@ -36,9 +36,9 @@
             <mu1>10.0</mu1>
             <mu2>10.0</mu2>
-            <!--<xacro:insert_block name="material" />-->
-<!--            <material>Gazebo/${material}</material>-->
+            <material>Gazebo/Black</material>
         </gazebo>
     </xacro:macro>
     <!-- Chassis Properties -->
+    <xacro:property name="chassis_mesh_path" value="package://robotics_configurations/alex_description/models/alex/meshes/ros_chassis_sw0001.stl"/>
     <xacro:property name="chassis_mass" value="0.1"/>
     <xacro:property name="chassis_width_x" value="0.192"/>
@@ -48,10 +48,20 @@
     <xacro:property name="chassis_iyy" value="${(chassis_mass / 12.0) * (chassis_width_x**2 + chassis_height_z**2)}"/>
     <xacro:property name="chassis_izz" value="${(chassis_mass / 12.0) * (chassis_width_x**2 + chassis_depth_y**2)}"/>
+    <xacro:property name="chassis_origin_z_offset" value="0.017475"/>
     <xacro:macro name="chassis_origin">
-        <origin xyz="0 ${-chassis_depth_y/2} 0" rpy="0 0 0"/>
+        <origin xyz="0 ${-chassis_depth_y/2 - chassis_origin_z_offset} 0" rpy="0 0 0"/>
     </xacro:macro>
     <xacro:macro name="chassis_joint_origin">
         <origin xyz="-0.068 0 0.056475" rpy="${pi/2} 0 ${-pi/2}"/>
     </xacro:macro>
+    <!-- * * * * * * * * * -->
+    <!-- Expansion Plate Properties -->
+    <xacro:property name="ep_mass" value="0.01"/>
+    <xacro:property name="ep_width_x" value="0.192"/>
+    <xacro:property name="ep_depth_y" value="0.059"/>
+    <xacro:property name="ep_height_z" value="0.276"/>
+    <xacro:property name="ep_ixx" value="${(ep_mass / 12.0) * (ep_depth_y**2 + ep_height_z**2)}"/>
+    <xacro:property name="ep_iyy" value="${(ep_mass / 12.0) * (ep_width_x**2 + ep_height_z**2)}"/>
+    <xacro:property name="ep_izz" value="${(ep_mass / 12.0) * (ep_width_x**2 + ep_depth_y**2)}"/>
     <!-- * * * * * * * * * -->
     <!-- Wheel Properties -->
@@ -62,12 +72,41 @@
     <xacro:property name="wheel_iyy" value="${wheel_ixx}"/>
     <xacro:property name="wheel_izz" value="${(chassis_mass * wheel_radius**2) / 2}"/>
+    <xacro:macro name="left_wheel_joint_origin">
+        <origin xyz="0 0.0805 0" rpy="${-pi/2} 0 0"/>
+    </xacro:macro>
     <xacro:macro name="right_wheel_joint_origin">
         <origin xyz="0 -0.0805 0" rpy="${-pi/2} 0 0"/>
     </xacro:macro>
-    <xacro:macro name="left_wheel_joint_origin">
-        <origin xyz="0 0.0805 0" rpy="${-pi/2} 0 0"/>
-    </xacro:macro>
-    <!-- * * * * * * * * * -->
-    <!-- Macros -->
+    <!-- * * * * * * * * * -->
+    <!-- Castor Properties -->
+    <xacro:property name="castor_mesh_path" value="package://robotics_configurations/alex_description/models/alex/meshes/castor_wheel_sw0001.stl"/>
+    <xacro:property name="castor_mass" value="0.001"/>
+    <xacro:property name="castor_height" value="0.025"/>
+    <xacro:property name="castor_radius" value="0.0162"/>
+    <xacro:property name="castor_ixx" value="${(castor_mass / 12.0) * (3 * castor_radius**2 + castor_height**2)}"/>
+    <xacro:property name="castor_iyy" value="${castor_ixx}"/>
+    <xacro:property name="castor_izz" value="${(castor_mass * castor_radius**2) / 2}"/>
+    <xacro:macro name="castor_mesh_origin">
+        <origin xyz="0.08 0 0.058515" rpy="${pi/2} 0 ${-pi/2}"/>
+    </xacro:macro>
+    <xacro:macro name="castor_collision_origin">
+        <origin xyz="0 0 ${-castor_height/2}" rpy="0 0 0"/>
+    </xacro:macro>
+    <xacro:macro name="castor_joint_origin">
+        <origin xyz="-0.148 0 -0.00204" rpy="0 0 0"/>
+    </xacro:macro>
+    <!-- * * * * * * * * * -->
+    <!-- Castor Wheel Properties -->
+    <xacro:property name="castor_wheel_mass" value="0.001"/>
+    <xacro:property name="castor_wheel_width" value="0.0145"/>
+    <xacro:property name="castor_wheel_radius" value="0.0125"/>
+    <xacro:property name="castor_wheel_ixx" value="${(castor_wheel_mass / 12.0) * (3 * castor_wheel_radius**2 + castor_wheel_width**2)}"/>
+    <xacro:property name="castor_wheel_iyy" value="${castor_wheel_ixx}"/>
+    <xacro:property name="castor_wheel_izz" value="${(castor_wheel_mass * castor_wheel_radius**2) / 2}"/>
+    <xacro:macro name="castor_wheel_joint_origin">
+        <origin xyz="-0.016 0 -0.0205" rpy="${-pi/2} 0 0"/>
+    </xacro:macro>
+    <!-- * * * * * * * * * -->
+    <!-- Generic Macros -->
     <xacro:macro name="x_axis">
         <axis xyz="1 0 0" rpy="0 0 0"/>
@@ -98,9 +137,10 @@
         </inertial>
         <visual>
-            <xacro:chassis_origin/>
-            <geometry>
-                <box size="${chassis_width_x} ${chassis_depth_y} ${chassis_height_z}"/>
-            </geometry>
-            <material name="grey"/>
+            <origin xyz="0 0 0" rpy="0 0 0"/>
+            <geometry>
+<!--                <box size="${chassis_width_x} ${chassis_depth_y} ${chassis_height_z}"/>-->
+                <mesh filename="${chassis_mesh_path}" scale="0.001 0.001 0.001"/>
+            </geometry>
+            <material name="black"/>
         </visual>
         <collision>
@@ -172,6 +212,56 @@
         <joint_properties damping="1.0" friction="1.0"/>
 	</joint>
-    <xacro:gazebo_params link_ref="left_wheel"/>
-    <xacro:gazebo_params link_ref="right_wheel"/>
+    <link name="castor">
+        <inertial>
+            <xacro:castor_collision_origin/>
+            <mass value="${castor_mass}"/>
+            <inertia ixx="${castor_ixx}" ixy="0.0" ixz="0.0" iyy="${castor_iyy}" iyz="0.0" izz="${castor_izz}"/>
+        </inertial>
+        <visual>
+            <xacro:castor_mesh_origin/>
+            <geometry>
+                <mesh filename="${castor_mesh_path}" scale="0.001 0.001 0.001"/>
+            </geometry>
+            <material name="grey"/>
+        </visual>
+        <collision>
+            <xacro:castor_collision_origin/>
+            <geometry>
+                <cylinder radius="${castor_radius}" length="${castor_height}"/>
+            </geometry>
+        </collision>
+    </link>
+    <joint name="baselink_castor_joint" type="continuous">
+    	<parent link="base_link"/>
+    	<child link="castor"/>
+    	<xacro:castor_joint_origin/>
+        <limit effort="1.0" velocity="0.45"/>
+        <xacro:z_axis/>
+        <joint_properties damping="1.0" friction="1.0"/>
+	</joint>
+    <link name="castor_wheel">
+        <inertial>
+            <origin rpy="0 0 0" xyz="0 0 0"/>
+            <mass value="${castor_wheel_mass}"/>
+            <inertia ixx="${castor_wheel_ixx}" ixy="0.0" ixz="0.0" iyy="${castor_wheel_iyy}" iyz="0.0" izz="${castor_wheel_izz}"/>
+        </inertial>
+        <collision>
+            <origin rpy="0 0 0" xyz="0 0 0"/>
+            <geometry>
+                <cylinder radius="${castor_wheel_radius}" length="${castor_wheel_width}"/>
+            </geometry>
+        </collision>
+    </link>
+    <joint name="castor_castorwheel_joint" type="continuous">
+    	<parent link="castor"/>
+    	<child link="castor_wheel"/>
+    	<xacro:castor_wheel_joint_origin/>
+        <limit effort="1.0" velocity="0.45"/>
+        <xacro:z_axis/>
+        <joint_properties damping="1.0" friction="1.0"/>
+	</joint>
+    <xacro:gazebo_wheel_params link_ref="left_wheel"/>
+    <xacro:gazebo_wheel_params link_ref="right_wheel"/>
+    <xacro:gazebo_wheel_params link_ref="castor_wheel"/>
     <!--<link name="castor_swivel">
     </link>
