Commit message: Add pan and tilt mechanisms

File: src/robotics_configurations/alex_description/robots/alex.urdf.xacro (robot description, xacro)
@@ -30,13 +30,4 @@
         </plugin>
     </gazebo>
-    <xacro:macro name="gazebo_wheel_params" params="link_ref">
-        <gazebo reference="${link_ref}">
-            <kp>100.0</kp>
-            <kd>100.0</kd>
-            <mu1>10.0</mu1>
-            <mu2>10.0</mu2>
-            <material>Gazebo/Black</material>
-        </gazebo>
-    </xacro:macro>
     <!-- Chassis Properties -->
     <xacro:property name="chassis_mesh_path" value="package://robotics_configurations/alex_description/models/alex/meshes/ros_chassis_sw0001.stl"/>
@@ -78,7 +69,17 @@
         <origin xyz="0 -0.0805 0" rpy="${-pi/2} 0 0"/>
     </xacro:macro>
+    <xacro:macro name="gazebo_wheel_params" params="link_ref">
+        <gazebo reference="${link_ref}">
+            <kp>500.0</kp>
+            <kd>500.0</kd>
+            <mu1>10.0</mu1>
+            <mu2>10.0</mu2>
+            <material>Gazebo/Black</material>
+        </gazebo>
+    </xacro:macro>
     <!-- * * * * * * * * * -->
     <!-- Castor Properties -->
-    <xacro:property name="castor_mesh_path" value="package://robotics_configurations/alex_description/models/alex/meshes/castor_wheel_sw0001.stl"/>
+    <xacro:property name="castor_mesh_path"
+                    value="package://robotics_configurations/alex_description/models/alex/meshes/castor_wheel_sw0001.stl"/>
     <xacro:property name="castor_mass" value="0.001"/>
     <xacro:property name="castor_height" value="0.025"/>
@@ -107,4 +108,47 @@
         <origin xyz="-0.016 0 -0.0205" rpy="${-pi/2} 0 0"/>
     </xacro:macro>
+    <xacro:macro name="gazebo_castor_wheel_params" params="link_ref">
+        <gazebo reference="${link_ref}">
+            <kp>1000.0</kp>
+            <kd>1000.0</kd>
+            <mu1>10.0</mu1>
+            <mu2>10.0</mu2>
+            <material>Gazebo/Black</material>
+        </gazebo>
+    </xacro:macro>
+    <!-- * * * * * * * * * -->
+    <!-- Pan Mechanism Properties -->
+    <xacro:property name="pan_mechanism_mesh_path"
+                    value="package://robotics_configurations/alex_description/models/alex/meshes/pan_servo_ros_sw0004.stl"/>
+    <xacro:property name="pan_mechanism_mass" value="0.005"/>
+    <xacro:property name="pan_mechanism_width_x" value="0.016"/>
+    <xacro:property name="pan_mechanism_depth_y" value="0.0385"/>
+    <xacro:property name="pan_mechanism_height_z" value="0.048"/>
+    <xacro:property name="pan_mechanism_ixx" value="${(pan_mechanism_mass / 12.0) * (pan_mechanism_depth_y**2 + pan_mechanism_height_z**2)}"/>
+    <xacro:property name="pan_mechanism_iyy" value="${(pan_mechanism_mass / 12.0) * (pan_mechanism_width_x**2 + pan_mechanism_height_z**2)}"/>
+    <xacro:property name="pan_mechanism_izz" value="${(pan_mechanism_mass / 12.0) * (pan_mechanism_width_x**2 + pan_mechanism_depth_y**2)}"/>
+    <xacro:macro name="pan_mechanism_origin">
+        <origin xyz="0 0 0" rpy="0 0 0"/>
+    </xacro:macro>
+    <xacro:macro name="pan_mechanism_joint_origin">
+        <origin xyz="0 -0.0372805 -0.142268" rpy="${pi} ${-pi/2} 0"/>
+    </xacro:macro>
+    <!-- * * * * * * * * * -->
+    <!-- Tilt Mechanism Properties -->
+<!--    <xacro:property name="tilt_mechanism_mesh_path"-->
+<!--                    value="package://robotics_configurations/alex_description/models/alex/meshes/pan_servo_ros_sw0004.stl"/>-->
+    <xacro:property name="tilt_mechanism_mass" value="0.005"/>
+    <xacro:property name="tilt_mechanism_width_x" value="0.016"/>
+    <xacro:property name="tilt_mechanism_depth_y" value="0.0385"/>
+    <xacro:property name="tilt_mechanism_height_z" value="0.048"/>
+    <xacro:property name="tilt_mechanism_ixx" value="${(tilt_mechanism_mass / 12.0) * (tilt_mechanism_depth_y**2 + tilt_mechanism_height_z**2)}"/>
+    <xacro:property name="tilt_mechanism_iyy" value="${(tilt_mechanism_mass / 12.0) * (tilt_mechanism_width_x**2 + tilt_mechanism_height_z**2)}"/>
+    <xacro:property name="tilt_mechanism_izz" value="${(tilt_mechanism_mass / 12.0) * (tilt_mechanism_width_x**2 + tilt_mechanism_depth_y**2)}"/>
+    <xacro:macro name="tilt_mechanism_origin">
+        <origin xyz="0 0 0" rpy="0 0 0"/>
+    </xacro:macro>
+    <xacro:macro name="tilt_mechanism_joint_origin">
+        <origin xyz="0 -0.04825 -0.000526152" rpy="${-pi/2} 0 ${pi}"/>
+    </xacro:macro>
     <!-- * * * * * * * * * -->
     <!-- Generic Macros -->
@@ -261,7 +305,67 @@
         <joint_properties damping="1.0" friction="1.0"/>
 	</joint>
+    <link name="pan_mechanism">
+        <inertial>
+            <xacro:pan_mechanism_origin/>
+            <mass value="${pan_mechanism_mass}"/>
+            <inertia ixx="${pan_mechanism_ixx}" ixy="0.0" ixz="0.0" iyy="${pan_mechanism_iyy}" iyz="0.0" izz="${pan_mechanism_izz}"/>
+        </inertial>
+        <visual>
+            <xacro:pan_mechanism_origin/>
+<!--            <origin rpy="0 0 0" xyz="0 0 0"/>-->
+            <geometry>
+                <box size="${pan_mechanism_width_x} ${pan_mechanism_depth_y} ${pan_mechanism_height_z}"/>
+<!--                <mesh filename="${pan_mechanism_mesh_path}" scale="0.001 0.001 0.001"/>-->
+            </geometry>
+            <material name="black"/>
+        </visual>
+        <collision>
+            <xacro:pan_mechanism_origin/>
+            <geometry>
+                <box size="${pan_mechanism_width_x} ${pan_mechanism_depth_y} ${pan_mechanism_height_z}"/>
+            </geometry>
+        </collision>
+    </link>
+    <joint name="pan_mechanism_joint" type="revolute">
+    	<parent link="chassis"/>
+    	<child link="pan_mechanism"/>
+    	<xacro:pan_mechanism_joint_origin/>
+        <limit lower="${-pi/2}" upper="${pi/2}" effort="1.0" velocity="${100*pi/180}"/>
+        <xacro:y_axis/>
+        <joint_properties damping="1.0" friction="1.0"/>
+	</joint>
+    <link name="tilt_mechanism">
+        <inertial>
+            <xacro:tilt_mechanism_origin/>
+            <mass value="${tilt_mechanism_mass}"/>
+            <inertia ixx="${tilt_mechanism_ixx}" ixy="0.0" ixz="0.0" iyy="${tilt_mechanism_iyy}" iyz="0.0" izz="${tilt_mechanism_izz}"/>
+        </inertial>
+        <visual>
+            <xacro:tilt_mechanism_origin/>
+<!--            <origin rpy="0 0 0" xyz="0 0 0"/>-->
+            <geometry>
+                <box size="${tilt_mechanism_width_x} ${tilt_mechanism_depth_y} ${tilt_mechanism_height_z}"/>
+<!--                <mesh filename="${tilt_mechanism_mesh_path}" scale="0.001 0.001 0.001"/>-->
+            </geometry>
+            <material name="black"/>
+        </visual>
+        <collision>
+            <xacro:tilt_mechanism_origin/>
+            <geometry>
+                <box size="${tilt_mechanism_width_x} ${tilt_mechanism_depth_y} ${tilt_mechanism_height_z}"/>
+            </geometry>
+        </collision>
+    </link>
+    <joint name="tilt_mechanism_joint" type="revolute">
+    	<parent link="pan_mechanism"/>
+    	<child link="tilt_mechanism"/>
+    	<xacro:tilt_mechanism_joint_origin/>
+        <limit lower="${-pi/2}" upper="${pi/2}" effort="1.0" velocity="${100*pi/180}"/>
+        <xacro:y_axis/>
+        <joint_properties damping="1.0" friction="1.0"/>
+	</joint>
     <xacro:gazebo_wheel_params link_ref="left_wheel"/>
     <xacro:gazebo_wheel_params link_ref="right_wheel"/>
-    <xacro:gazebo_wheel_params link_ref="castor_wheel"/>
+    <xacro:gazebo_castor_wheel_params link_ref="castor_wheel"/>
     <!--<link name="castor_swivel">
     </link>

Commit message: Add new chassis mesh and add servo meshes

File: src/robotics_configurations/alex_description/robots/alex.urdf.xacro (robot description, xacro)
@@ -31,5 +31,6 @@
     </gazebo>
     <!-- Chassis Properties -->
-    <xacro:property name="chassis_mesh_path" value="package://robotics_configurations/alex_description/models/alex/meshes/ros_chassis_sw0001.stl"/>
+    <xacro:property name="chassis_mesh_path"
+                    value="package://robotics_configurations/alex_description/models/alex/meshes/ros_chassis_sw0002.stl"/>
     <xacro:property name="chassis_mass" value="0.1"/>
     <xacro:property name="chassis_width_x" value="0.192"/>
@@ -134,8 +135,17 @@
         <origin xyz="0 -0.0372805 -0.142268" rpy="${pi} ${-pi/2} 0"/>
     </xacro:macro>
+    <xacro:macro name="servo_params" params="link_ref">
+        <gazebo reference="${link_ref}">
+            <kp>10000.0</kp>
+            <kd>10000.0</kd>
+            <mu1>1.0</mu1>
+            <mu2>1.0</mu2>
+            <material>Gazebo/Black</material>
+        </gazebo>
+    </xacro:macro>
     <!-- * * * * * * * * * -->
     <!-- Tilt Mechanism Properties -->
-<!--    <xacro:property name="tilt_mechanism_mesh_path"-->
-<!--                    value="package://robotics_configurations/alex_description/models/alex/meshes/pan_servo_ros_sw0004.stl"/>-->
+    <xacro:property name="tilt_mechanism_mesh_path"
+                    value="package://robotics_configurations/alex_description/models/alex/meshes/tilt_servo_ros_sw0002.stl"/>
     <xacro:property name="tilt_mechanism_mass" value="0.005"/>
     <xacro:property name="tilt_mechanism_width_x" value="0.016"/>
@@ -149,5 +159,5 @@
     </xacro:macro>
     <xacro:macro name="tilt_mechanism_joint_origin">
-        <origin xyz="0 -0.04825 -0.000526152" rpy="${-pi/2} 0 ${pi}"/>
+        <origin xyz="0 -0.04825 -0.000526152" rpy="${pi/2} 0 ${pi}"/>
     </xacro:macro>
     <!-- * * * * * * * * * -->
@@ -312,9 +322,9 @@
         </inertial>
         <visual>
-            <xacro:pan_mechanism_origin/>
-<!--            <origin rpy="0 0 0" xyz="0 0 0"/>-->
-            <geometry>
-                <box size="${pan_mechanism_width_x} ${pan_mechanism_depth_y} ${pan_mechanism_height_z}"/>
-<!--                <mesh filename="${pan_mechanism_mesh_path}" scale="0.001 0.001 0.001"/>-->
+<!--            <xacro:pan_mechanism_origin/>-->
+            <origin rpy="0 0 0" xyz="0 0 0"/>
+            <geometry>
+<!--                <box size="${pan_mechanism_width_x} ${pan_mechanism_depth_y} ${pan_mechanism_height_z}"/>-->
+                <mesh filename="${pan_mechanism_mesh_path}" scale="0.001 0.001 0.001"/>
             </geometry>
             <material name="black"/>
@@ -342,9 +352,9 @@
         </inertial>
         <visual>
-            <xacro:tilt_mechanism_origin/>
-<!--            <origin rpy="0 0 0" xyz="0 0 0"/>-->
-            <geometry>
-                <box size="${tilt_mechanism_width_x} ${tilt_mechanism_depth_y} ${tilt_mechanism_height_z}"/>
-<!--                <mesh filename="${tilt_mechanism_mesh_path}" scale="0.001 0.001 0.001"/>-->
+<!--            <xacro:tilt_mechanism_origin/>-->
+            <origin rpy="0 0 0" xyz="0 0 0"/>
+            <geometry>
+<!--                <box size="${tilt_mechanism_width_x} ${tilt_mechanism_depth_y} ${tilt_mechanism_height_z}"/>-->
+                <mesh filename="${tilt_mechanism_mesh_path}" scale="0.001 0.001 0.001"/>
             </geometry>
             <material name="black"/>
@@ -368,4 +378,6 @@
     <xacro:gazebo_wheel_params link_ref="right_wheel"/>
     <xacro:gazebo_castor_wheel_params link_ref="castor_wheel"/>
+    <xacro:servo_params link_ref="pan_mechanism"/>
+    <xacro:servo_params link_ref="tilt_mechanism"/>
     <!--<link name="castor_swivel">
     </link>

Commit message: Add wheel meshes

File: src/robotics_configurations/alex_description/robots/alex.urdf.xacro (robot description, xacro)
@@ -58,4 +58,6 @@
     <!-- * * * * * * * * * -->
     <!-- Wheel Properties -->
+    <xacro:property name="wheel_mesh_path"
+                    value="package://robotics_configurations/alex_description/models/alex/meshes/ros_wheel_sw0002.stl"/>
     <xacro:property name="wheel_mass" value="0.01"/>
     <xacro:property name="wheel_width" value="0.029"/>
@@ -64,6 +66,12 @@
     <xacro:property name="wheel_iyy" value="${wheel_ixx}"/>
     <xacro:property name="wheel_izz" value="${(chassis_mass * wheel_radius**2) / 2}"/>
+    <xacro:macro name="left_wheel_mesh_origin">
+        <origin xyz="0 0 0" rpy="${pi/2} ${pi} 0"/>
+    </xacro:macro>
     <xacro:macro name="left_wheel_joint_origin">
         <origin xyz="0 0.0805 0" rpy="${-pi/2} 0 0"/>
+    </xacro:macro>
+    <xacro:macro name="right_wheel_mesh_origin">
+        <origin xyz="0 0 0" rpy="${pi/2} 0 0"/>
     </xacro:macro>
     <xacro:macro name="right_wheel_joint_origin">
@@ -217,7 +225,8 @@
         </inertial>
         <visual>
-            <origin rpy="0 0 0" xyz="0 0 0"/>
-            <geometry>
-                <cylinder radius="${wheel_radius}" length="${wheel_width}"/>
+            <xacro:right_wheel_mesh_origin/>
+            <geometry>
+                <mesh filename="${wheel_mesh_path}" scale="0.001 0.001 0.001"/>
+<!--                <cylinder radius="${wheel_radius}" length="${wheel_width}"/>-->
             </geometry>
             <material name="black"/>
@@ -245,7 +254,8 @@
         </inertial>
         <visual>
-            <origin rpy="0 0 0" xyz="0 0 0"/>
-            <geometry>
-                <cylinder radius="${wheel_radius}" length="${wheel_width}"/>
+            <xacro:left_wheel_mesh_origin/>
+            <geometry>
+                <mesh filename="${wheel_mesh_path}" scale="0.001 0.001 0.001"/>
+<!--                <cylinder radius="${wheel_radius}" length="${wheel_width}"/>-->
             </geometry>
             <material name="black"/>

Commit message: Change colours

File: src/robotics_configurations/alex_description/robots/alex.urdf.xacro (robot description, xacro)
@@ -21,5 +21,5 @@
             <leftJoint>baselink_left_wheel_joint</leftJoint>
             <rightJoint>baselink_right_wheel_joint</rightJoint>
-            <wheelSeparation>0.0175</wheelSeparation>
+            <wheelSeparation>0.175</wheelSeparation>
             <wheelDiameter>0.075</wheelDiameter>
             <torque>0.01</torque>
@@ -84,5 +84,5 @@
             <mu1>10.0</mu1>
             <mu2>10.0</mu2>
-            <material>Gazebo/Black</material>
+            <material>Gazebo/FlatBlack</material>
         </gazebo>
     </xacro:macro>
@@ -123,5 +123,5 @@
             <mu1>10.0</mu1>
             <mu2>10.0</mu2>
-            <material>Gazebo/Black</material>
+            <material>Gazebo/FlatBlack</material>
         </gazebo>
     </xacro:macro>
@@ -149,5 +149,5 @@
             <mu1>1.0</mu1>
             <mu2>1.0</mu2>
-            <material>Gazebo/Black</material>
+            <material>Gazebo/FlatBlack</material>
         </gazebo>
     </xacro:macro>
@@ -218,4 +218,11 @@
     	<xacro:chassis_joint_origin/>
 	</joint>
+    <gazebo reference="chassis">
+        <kp>10000.0</kp>
+        <kd>10000.0</kd>
+        <mu1>1.0</mu1>
+        <mu2>1.0</mu2>
+        <material>Gazebo/FlatBlack</material>
+    </gazebo>
     <link name="right_wheel">
         <inertial>
@@ -304,4 +311,11 @@
         <joint_properties damping="1.0" friction="1.0"/>
 	</joint>
+    <gazebo reference="castor">
+        <kp>10000.0</kp>
+        <kd>10000.0</kd>
+        <mu1>10.0</mu1>
+        <mu2>10.0</mu2>
+        <material>Gazebo/Grey</material>
+    </gazebo>
     <link name="castor_wheel">
         <inertial>

Commit message: Add servo position control, camera and camera meshes

File: src/robotics_configurations/alex_description/robots/alex.urdf.xacro (robot description, xacro)
@@ -29,4 +29,7 @@
             <robotBaseFrame>base_link</robotBaseFrame>
         </plugin>
+        <plugin name="gazebo_ros_control" filename="libgazebo_ros_control.so">
+            <robotNamespace>/alex</robotNamespace>
+        </plugin>
     </gazebo>
     <!-- Chassis Properties -->
@@ -170,4 +173,30 @@
     </xacro:macro>
     <!-- * * * * * * * * * -->
+    <!-- Camera Module Properties -->
+    <xacro:property name="camera_module_mesh_path"
+                    value="package://robotics_configurations/alex_description/models/alex/meshes/camera_module_sw0001.stl"/>
+    <xacro:property name="camera_module_mass" value="0.005"/>
+    <xacro:property name="camera_module_width_x" value="0.02375"/>
+    <xacro:property name="camera_module_depth_y" value="0.0124"/>
+    <xacro:property name="camera_module_height_z" value="0.02375"/>
+    <xacro:property name="camera_module_ixx" value="${(camera_module_mass / 12.0) * (camera_module_depth_y**2 + camera_module_height_z**2)}"/>
+    <xacro:property name="camera_module_iyy" value="${(camera_module_mass / 12.0) * (camera_module_width_x**2 + camera_module_height_z**2)}"/>
+    <xacro:property name="camera_module_izz" value="${(camera_module_mass / 12.0) * (camera_module_width_x**2 + camera_module_depth_y**2)}"/>
+    <xacro:property name="camera_module_collision_y_offset" value="-0.0031"/>
+    <xacro:macro name="camera_module_box_origin">
+        <origin xyz="0 ${camera_module_collision_y_offset} 0" rpy="0 0 0"/>
+    </xacro:macro>
+    <xacro:macro name="camera_module_joint_origin">
+        <origin xyz="0.0176 0.00035 0" rpy="0 0 ${-pi/2}"/>
+    </xacro:macro>
+    <!-- Camera Sensor Properties -->
+<!--    <xacro:macro name="camera_sensor_joint_origin">-->
+<!--        <origin xyz="0 0.0014 0" rpy="${-pi/2} ${pi} 0"/>-->
+<!--    </xacro:macro>-->
+    <xacro:macro name="camera_sensor_joint_origin">
+        <origin xyz="0 0.0014 0" rpy="${pi} 0 ${pi/2}"/>
+    </xacro:macro>
+    <xacro:property name="camera_hfov_rad" value="${108*pi/180}"/>
+    <!-- * * * * * * * * * -->
     <!-- Generic Macros -->
     <xacro:macro name="x_axis">
@@ -185,5 +214,5 @@
         <pose>0 0 ${wheel_radius} 0 0 0</pose>
         <visual>
-            <origin rpy="0.0 0 0" xyz="0 0 0"/>
+            <origin rpy="0 0 0" xyz="0 0 0"/>
             <geometry>
                 <box size="0.01 0.01 0.01"/>
@@ -404,9 +433,98 @@
     <xacro:servo_params link_ref="pan_mechanism"/>
     <xacro:servo_params link_ref="tilt_mechanism"/>
-    <!--<link name="castor_swivel">
-    </link>
-    <link name="castor_wheel">
-    </link>
-    <link name="chassis">
-    </link>-->
+    <xacro:macro name="servo_transmission_macro" params="joint servo_type">
+        <transmission name="${servo_type}_transmission">
+            <type>transmission_interface/SimpleTransmission</type>
+            <joint name="${joint}">
+                <hardwareInterface>hardware_interface/PositionJointInterface</hardwareInterface>
+            </joint>
+            <actuator name="${servo_type}_servo_actuator">
+                <hardwareInterface>hardware_interface/PositionJointInterface</hardwareInterface>
+                <mechanicalReduction>1</mechanicalReduction>
+            </actuator>
+        </transmission>
+    </xacro:macro>
+    <xacro:servo_transmission_macro joint="pan_mechanism_joint" servo_type="pan" />
+    <xacro:servo_transmission_macro joint="tilt_mechanism_joint" servo_type="tilt" />
+    <link name="camera_module">
+        <inertial>
+            <xacro:camera_module_box_origin/>
+            <mass value="${camera_module_mass}"/>
+            <inertia ixx="${camera_module_ixx}" ixy="0.0" ixz="0.0" iyy="${camera_module_iyy}" iyz="0.0" izz="${camera_module_izz}"/>
+        </inertial>
+        <visual>
+<!--            <xacro:camera_module_box_origin/>-->
+            <origin rpy="0 0 0" xyz="0 0 0"/>
+            <geometry>
+<!--                <box size="${camera_module_width_x} ${camera_module_depth_y} ${camera_module_height_z}"/>-->
+                <mesh filename="${camera_module_mesh_path}" scale="0.001 0.001 0.001"/>
+            </geometry>
+            <material name="black"/>
+        </visual>
+        <collision>
+            <xacro:camera_module_box_origin/>
+            <geometry>
+                <box size="${camera_module_width_x} ${camera_module_depth_y} ${camera_module_height_z}"/>
+            </geometry>
+        </collision>
+    </link>
+    <joint name="camera_module_joint" type="fixed">
+    	<parent link="tilt_mechanism"/>
+    	<child link="camera_module"/>
+    	<xacro:camera_module_joint_origin/>
+	</joint>
+    <link name="camera_sensor">
+        <visual>
+            <origin rpy="0 0 0" xyz="0 0 0"/>
+            <geometry>
+                <box size="0.001 0.001 0.001"/>
+            </geometry>
+            <material name="red"/>
+        </visual>
+    </link>
+    <joint name="camera_sensor_joint" type="fixed">
+    	<parent link="camera_module"/>
+    	<child link="camera_sensor"/>
+    	<xacro:camera_sensor_joint_origin/>
+	</joint>
+    <!-- camera -->
+    <gazebo reference="camera_sensor">
+        <sensor type="camera" name="camera1">
+            <update_rate>30.0</update_rate>
+            <camera name="pan_tilt_camera">
+                <horizontal_fov>${camera_hfov_rad}</horizontal_fov>
+                <image>
+                    <width>640</width>
+                    <height>480</height>
+                    <format>R8G8B8</format>
+                </image>
+                <clip>
+                    <near>0.02</near>
+                    <far>300</far>
+                </clip>
+                <noise>
+                    <type>gaussian</type>
+                    <!-- Noise is sampled independently per pixel on each frame.
+                    That pixel's noise value is added to each of its color
+                    channels, which at that point lie in the range [0,1]. -->
+                    <mean>0.0</mean>
+                    <stddev>0.007</stddev>
+                </noise>
+            </camera>
+            <plugin name="camera_controller" filename="libgazebo_ros_camera.so">
+                <alwaysOn>true</alwaysOn>
+                <updateRate>0.0</updateRate>
+                <cameraName>alex/camera1</cameraName>
+                <imageTopicName>image_raw</imageTopicName>
+                <cameraInfoTopicName>camera_info</cameraInfoTopicName>
+                <frameName>camera_sensor</frameName>
+                <hackBaseline>0.07</hackBaseline>
+                <distortionK1>0.0</distortionK1>
+                <distortionK2>0.0</distortionK2>
+                <distortionK3>0.0</distortionK3>
+                <distortionT1>0.0</distortionT1>
+                <distortionT2>0.0</distortionT2>
+            </plugin>
+        </sensor>
+    </gazebo>
 </robot>
