Commit message: Add new meshes with proper colours and change directory of meshes

File: src/robotics_configurations/alex_description/robots/alex.urdf.xacro (robot description, xacro)
@@ -35,5 +35,5 @@
     <!-- Chassis Properties -->
     <xacro:property name="chassis_mesh_path"
-                    value="package://alex_description/models/alex/meshes/ros_chassis_sw0002.stl"/>
+                    value="package://alex_description/models/chassis_asm.dae"/>
     <xacro:property name="chassis_mass" value="0.1"/>
     <xacro:property name="chassis_width_x" value="0.192"/>
@@ -62,5 +62,5 @@
     <!-- Wheel Properties -->
     <xacro:property name="wheel_mesh_path"
-                    value="package://alex_description/models/alex/meshes/ros_wheel_sw0002.stl"/>
+                    value="package://alex_description/models/wheel_asm.dae"/>
     <xacro:property name="wheel_mass" value="0.01"/>
     <xacro:property name="wheel_width" value="0.029"/>
@@ -70,5 +70,5 @@
     <xacro:property name="wheel_izz" value="${(chassis_mass * wheel_radius**2) / 2}"/>
     <xacro:macro name="left_wheel_mesh_origin">
-        <origin xyz="0 0 0" rpy="${pi/2} ${pi} 0"/>
+        <origin xyz="0 0 0" rpy="0 ${pi} 0"/>
     </xacro:macro>
     <xacro:macro name="left_wheel_joint_origin">
@@ -76,5 +76,5 @@
     </xacro:macro>
     <xacro:macro name="right_wheel_mesh_origin">
-        <origin xyz="0 0 0" rpy="${pi/2} 0 0"/>
+        <origin xyz="0 0 0" rpy="0 0 0"/>
     </xacro:macro>
     <xacro:macro name="right_wheel_joint_origin">
@@ -87,5 +87,5 @@
             <mu1>10.0</mu1>
             <mu2>10.0</mu2>
-            <material>Gazebo/FlatBlack</material>
+<!--            <material>Gazebo/FlatBlack</material>-->
         </gazebo>
     </xacro:macro>
@@ -93,5 +93,5 @@
     <!-- Castor Properties -->
     <xacro:property name="castor_mesh_path"
-                    value="package://alex_description/models/alex/meshes/castor_wheel_sw0001.stl"/>
+                    value="package://alex_description/models/castor_wheel_sw0001.stl"/>
     <xacro:property name="castor_mass" value="0.001"/>
     <xacro:property name="castor_height" value="0.025"/>
@@ -132,5 +132,5 @@
     <!-- Pan Mechanism Properties -->
     <xacro:property name="pan_mechanism_mesh_path"
-                    value="package://alex_description/models/alex/meshes/pan_servo_ros_sw0004.stl"/>
+                    value="package://alex_description/models/pan_servo_ros_sw0004.stl"/>
     <xacro:property name="pan_mechanism_mass" value="0.005"/>
     <xacro:property name="pan_mechanism_width_x" value="0.016"/>
@@ -158,5 +158,5 @@
     <!-- Tilt Mechanism Properties -->
     <xacro:property name="tilt_mechanism_mesh_path"
-                    value="package://alex_description/models/alex/meshes/tilt_servo_ros_sw0002.stl"/>
+                    value="package://alex_description/models/tilt_servo_ros_sw0002.stl"/>
     <xacro:property name="tilt_mechanism_mass" value="0.005"/>
     <xacro:property name="tilt_mechanism_width_x" value="0.016"/>
@@ -175,5 +175,5 @@
     <!-- Camera Module Properties -->
     <xacro:property name="camera_module_mesh_path"
-                    value="package://alex_description/models/alex/meshes/camera_module_sw0001.stl"/>
+                    value="package://alex_description/models/camera_module_sw0001.stl"/>
     <xacro:property name="camera_module_mass" value="0.005"/>
     <xacro:property name="camera_module_width_x" value="0.02375"/>
@@ -231,5 +231,5 @@
             <geometry>
 <!--                <box size="${chassis_width_x} ${chassis_depth_y} ${chassis_height_z}"/>-->
-                <mesh filename="${chassis_mesh_path}" scale="0.001 0.001 0.001"/>
+                <mesh filename="${chassis_mesh_path}"/>
             </geometry>
             <material name="black"/>
@@ -252,5 +252,5 @@
         <mu1>1.0</mu1>
         <mu2>1.0</mu2>
-        <material>Gazebo/FlatBlack</material>
+<!--        <material>Gazebo/FlatBlack</material>-->
     </gazebo>
     <link name="right_wheel">
@@ -263,5 +263,5 @@
             <xacro:right_wheel_mesh_origin/>
             <geometry>
-                <mesh filename="${wheel_mesh_path}" scale="0.001 0.001 0.001"/>
+                <mesh filename="${wheel_mesh_path}"/>
 <!--                <cylinder radius="${wheel_radius}" length="${wheel_width}"/>-->
             </geometry>
@@ -292,5 +292,5 @@
             <xacro:left_wheel_mesh_origin/>
             <geometry>
-                <mesh filename="${wheel_mesh_path}" scale="0.001 0.001 0.001"/>
+                <mesh filename="${wheel_mesh_path}"/>
 <!--                <cylinder radius="${wheel_radius}" length="${wheel_width}"/>-->
             </geometry>

Commit message: Add ep, pt4 and servo daes

File: src/robotics_configurations/alex_description/robots/alex.urdf.xacro (robot description, xacro)
@@ -52,11 +52,31 @@
     <!-- * * * * * * * * * -->
     <!-- Expansion Plate Properties -->
-    <xacro:property name="ep_mass" value="0.01"/>
-    <xacro:property name="ep_width_x" value="0.192"/>
-    <xacro:property name="ep_depth_y" value="0.059"/>
-    <xacro:property name="ep_height_z" value="0.276"/>
+    <xacro:property name="ep_mesh_path"
+                    value="package://alex_description/models/EP_asm.dae"/>
+    <xacro:property name="ep_mass" value="0.05"/>
+    <xacro:property name="ep_width_x" value="0.1015"/>
+    <xacro:property name="ep_depth_y" value="0.018"/>
+    <xacro:property name="ep_height_z" value="0.134"/>
     <xacro:property name="ep_ixx" value="${(ep_mass / 12.0) * (ep_depth_y**2 + ep_height_z**2)}"/>
     <xacro:property name="ep_iyy" value="${(ep_mass / 12.0) * (ep_width_x**2 + ep_height_z**2)}"/>
     <xacro:property name="ep_izz" value="${(ep_mass / 12.0) * (ep_width_x**2 + ep_depth_y**2)}"/>
+    <xacro:property name="ep_origin_y_offset" value="0.0085"/>
+    <xacro:macro name="ep_box_origin">
+        <origin xyz="0 -${ep_origin_y_offset} 0" rpy="0 0 0"/>
+    </xacro:macro>
+    <!-- * * * * * * * * * -->
+    <!-- pi-top [4] Properties -->
+    <xacro:property name="pt4_mesh_path"
+                    value="package://alex_description/models/4_asm.dae"/>
+    <xacro:property name="pt4_mass" value="0.3"/>
+    <xacro:property name="pt4_width_x" value="0.0995"/>
+    <xacro:property name="pt4_depth_y" value="0.034"/>
+    <xacro:property name="pt4_height_z" value="0.132"/>
+    <xacro:property name="pt4_ixx" value="${(pt4_mass / 12.0) * (pt4_depth_y**2 + pt4_height_z**2)}"/>
+    <xacro:property name="pt4_iyy" value="${(pt4_mass / 12.0) * (pt4_width_x**2 + pt4_height_z**2)}"/>
+    <xacro:property name="pt4_izz" value="${(pt4_mass / 12.0) * (pt4_width_x**2 + pt4_depth_y**2)}"/>
+    <xacro:macro name="pt4_box_origin">
+        <origin xyz="0 ${pt4_depth_y/2} 0" rpy="0 0 0"/>
+    </xacro:macro>
     <!-- * * * * * * * * * -->
     <!-- Wheel Properties -->
@@ -132,5 +152,5 @@
     <!-- Pan Mechanism Properties -->
     <xacro:property name="pan_mechanism_mesh_path"
-                    value="package://alex_description/models/pan_servo_ros_sw0004.stl"/>
+                    value="package://alex_description/models/pan_asm_2.dae"/>
     <xacro:property name="pan_mechanism_mass" value="0.005"/>
     <xacro:property name="pan_mechanism_width_x" value="0.016"/>
@@ -152,5 +172,4 @@
             <mu1>1.0</mu1>
             <mu2>1.0</mu2>
-            <material>Gazebo/FlatBlack</material>
         </gazebo>
     </xacro:macro>
@@ -254,4 +273,70 @@
 <!--        <material>Gazebo/FlatBlack</material>-->
     </gazebo>
+    <link name="ep">
+        <inertial>
+            <xacro:ep_box_origin/>
+            <mass value="${ep_mass}"/>
+            <inertia ixx="${ep_ixx}" ixy="0.0" ixz="0.0" iyy="${ep_iyy}" iyz="0.0" izz="${ep_izz}"/>
+        </inertial>
+        <visual>
+            <origin xyz="0 0 0" rpy="0 0 0"/>
+            <geometry>
+<!--                <box size="${ep_width_x} ${ep_depth_y} ${ep_height_z}"/>-->
+                <mesh filename="${ep_mesh_path}"/>
+            </geometry>
+            <material name="black"/>
+        </visual>
+        <collision>
+            <xacro:ep_box_origin/>
+            <geometry>
+                <box size="${ep_width_x} ${ep_depth_y} ${ep_height_z}"/>
+            </geometry>
+        </collision>
+    </link>
+    <joint name="chassis_ep_joint" type="fixed">
+    	<parent link="chassis"/>
+    	<child link="ep"/>
+<!--    	<xacro:ep_joint_origin/>-->
+	</joint>
+    <gazebo reference="ep">
+        <kp>10000.0</kp>
+        <kd>10000.0</kd>
+        <mu1>1.0</mu1>
+        <mu2>1.0</mu2>
+<!--        <material>Gazebo/FlatBlack</material>-->
+    </gazebo>
+    <link name="pt4">
+        <inertial>
+            <xacro:pt4_box_origin/>
+            <mass value="${pt4_mass}"/>
+            <inertia ixx="${pt4_ixx}" ixy="0.0" ixz="0.0" iyy="${pt4_iyy}" iyz="0.0" izz="${pt4_izz}"/>
+        </inertial>
+        <visual>
+            <origin xyz="0 0 0" rpy="0 0 0"/>
+            <geometry>
+<!--                <box size="${pt4_width_x} ${pt4_depth_y} ${pt4_height_z}"/>-->
+                <mesh filename="${pt4_mesh_path}"/>
+            </geometry>
+            <material name="black"/>
+        </visual>
+        <collision>
+            <xacro:pt4_box_origin/>
+            <geometry>
+                <box size="${pt4_width_x} ${pt4_depth_y} ${pt4_height_z}"/>
+            </geometry>
+        </collision>
+    </link>
+    <joint name="chassis_pt4_joint" type="fixed">
+    	<parent link="chassis"/>
+    	<child link="pt4"/>
+<!--    	<xacro:pt4_joint_origin/>-->
+	</joint>
+    <gazebo reference="pt4">
+        <kp>10000.0</kp>
+        <kd>10000.0</kd>
+        <mu1>1.0</mu1>
+        <mu2>1.0</mu2>
+<!--        <material>Gazebo/FlatBlack</material>-->
+    </gazebo>
     <link name="right_wheel">
         <inertial>
@@ -379,5 +464,5 @@
             <geometry>
 <!--                <box size="${pan_mechanism_width_x} ${pan_mechanism_depth_y} ${pan_mechanism_height_z}"/>-->
-                <mesh filename="${pan_mechanism_mesh_path}" scale="0.001 0.001 0.001"/>
+                <mesh filename="${pan_mechanism_mesh_path}"/>
             </geometry>
             <material name="black"/>

Commit message: add camera, tilt and update pt4 (dae)

File: src/robotics_configurations/alex_description/robots/alex.urdf.xacro (robot description, xacro)
@@ -68,5 +68,5 @@
     <!-- pi-top [4] Properties -->
     <xacro:property name="pt4_mesh_path"
-                    value="package://alex_description/models/4_asm.dae"/>
+                    value="package://alex_description/models/4_asm_2.dae"/>
     <xacro:property name="pt4_mass" value="0.3"/>
     <xacro:property name="pt4_width_x" value="0.0995"/>
@@ -107,5 +107,4 @@
             <mu1>10.0</mu1>
             <mu2>10.0</mu2>
-<!--            <material>Gazebo/FlatBlack</material>-->
         </gazebo>
     </xacro:macro>
@@ -146,5 +145,4 @@
             <mu1>10.0</mu1>
             <mu2>10.0</mu2>
-            <material>Gazebo/FlatBlack</material>
         </gazebo>
     </xacro:macro>
@@ -177,5 +175,5 @@
     <!-- Tilt Mechanism Properties -->
     <xacro:property name="tilt_mechanism_mesh_path"
-                    value="package://alex_description/models/tilt_servo_ros_sw0002.stl"/>
+                    value="package://alex_description/models/tilt_asm.dae"/>
     <xacro:property name="tilt_mechanism_mass" value="0.005"/>
     <xacro:property name="tilt_mechanism_width_x" value="0.016"/>
@@ -194,5 +192,5 @@
     <!-- Camera Module Properties -->
     <xacro:property name="camera_module_mesh_path"
-                    value="package://alex_description/models/camera_module_sw0001.stl"/>
+                    value="package://alex_description/models/camera_asm.dae"/>
     <xacro:property name="camera_module_mass" value="0.005"/>
     <xacro:property name="camera_module_width_x" value="0.02375"/>
@@ -271,5 +269,4 @@
         <mu1>1.0</mu1>
         <mu2>1.0</mu2>
-<!--        <material>Gazebo/FlatBlack</material>-->
     </gazebo>
     <link name="ep">
@@ -304,5 +301,4 @@
         <mu1>1.0</mu1>
         <mu2>1.0</mu2>
-<!--        <material>Gazebo/FlatBlack</material>-->
     </gazebo>
     <link name="pt4">
@@ -337,5 +333,4 @@
         <mu1>1.0</mu1>
         <mu2>1.0</mu2>
-<!--        <material>Gazebo/FlatBlack</material>-->
     </gazebo>
     <link name="right_wheel">
@@ -406,5 +401,5 @@
             <xacro:castor_mesh_origin/>
             <geometry>
-                <mesh filename="${castor_mesh_path}" scale="0.001 0.001 0.001"/>
+                <mesh filename="${castor_mesh_path}"/>
             </geometry>
             <material name="grey"/>
@@ -494,5 +489,5 @@
             <geometry>
 <!--                <box size="${tilt_mechanism_width_x} ${tilt_mechanism_depth_y} ${tilt_mechanism_height_z}"/>-->
-                <mesh filename="${tilt_mechanism_mesh_path}" scale="0.001 0.001 0.001"/>
+                <mesh filename="${tilt_mechanism_mesh_path}"/>
             </geometry>
             <material name="black"/>
@@ -543,5 +538,5 @@
             <geometry>
 <!--                <box size="${camera_module_width_x} ${camera_module_depth_y} ${camera_module_height_z}"/>-->
-                <mesh filename="${camera_module_mesh_path}" scale="0.001 0.001 0.001"/>
+                <mesh filename="${camera_module_mesh_path}"/>
             </geometry>
             <material name="black"/>

Commit message: delete unused stls

File: src/robotics_configurations/alex_description/robots/alex.urdf.xacro (robot description, xacro)
@@ -112,5 +112,5 @@
     <!-- Castor Properties -->
     <xacro:property name="castor_mesh_path"
-                    value="package://alex_description/models/castor_wheel_sw0001.stl"/>
+                    value="package://alex_description/models/castor_asm_3.dae"/>
     <xacro:property name="castor_mass" value="0.001"/>
     <xacro:property name="castor_height" value="0.025"/>
@@ -403,5 +403,4 @@
                 <mesh filename="${castor_mesh_path}"/>
             </geometry>
-            <material name="grey"/>
         </visual>
         <collision>
@@ -425,5 +424,4 @@
         <mu1>10.0</mu1>
         <mu2>10.0</mu2>
-        <material>Gazebo/Grey</material>
     </gazebo>
     <link name="castor_wheel">

Commit message: Update for gzweb compatability with SDFs and model dirs

File: src/robotics_configurations/alex_description/robots/alex.urdf.xacro (robot description, xacro)
@@ -35,6 +35,6 @@
     <!-- Chassis Properties -->
     <xacro:property name="chassis_mesh_path"
-                    value="package://alex_description/models/chassis_asm.dae"/>
-    <xacro:property name="chassis_mass" value="0.1"/>
+                    value="model://alex/meshes/chassis_asm.dae"/>
+    <xacro:property name="chassis_mass" value="0.650"/>
     <xacro:property name="chassis_width_x" value="0.192"/>
     <xacro:property name="chassis_depth_y" value="0.059"/>
@@ -53,5 +53,5 @@
     <!-- Expansion Plate Properties -->
     <xacro:property name="ep_mesh_path"
-                    value="package://alex_description/models/EP_asm.dae"/>
+                    value="model://alex/meshes/EP_asm.dae"/>
     <xacro:property name="ep_mass" value="0.05"/>
     <xacro:property name="ep_width_x" value="0.1015"/>
@@ -68,6 +68,6 @@
     <!-- pi-top [4] Properties -->
     <xacro:property name="pt4_mesh_path"
-                    value="package://alex_description/models/4_asm_2.dae"/>
-    <xacro:property name="pt4_mass" value="0.3"/>
+                    value="model://alex/meshes/4_asm_2.dae"/>
+    <xacro:property name="pt4_mass" value="0.390"/>
     <xacro:property name="pt4_width_x" value="0.0995"/>
     <xacro:property name="pt4_depth_y" value="0.034"/>
@@ -82,5 +82,5 @@
     <!-- Wheel Properties -->
     <xacro:property name="wheel_mesh_path"
-                    value="package://alex_description/models/wheel_asm.dae"/>
+                    value="model://alex/meshes/wheel_asm.dae"/>
     <xacro:property name="wheel_mass" value="0.01"/>
     <xacro:property name="wheel_width" value="0.029"/>
@@ -101,4 +101,8 @@
         <origin xyz="0 -0.0805 0" rpy="${-pi/2} 0 0"/>
     </xacro:macro>
+    <xacro:property name="wheel_effort" value="" />
+    <xacro:property name="wheel_damping" value="" />
+    <xacro:property name="wheel_friction" value="" />
+    <xacro:property name="wheel_velocity" value="" />
     <xacro:macro name="gazebo_wheel_params" params="link_ref">
         <gazebo reference="${link_ref}">
@@ -112,5 +116,5 @@
     <!-- Castor Properties -->
     <xacro:property name="castor_mesh_path"
-                    value="package://alex_description/models/castor_asm_3.dae"/>
+                    value="model://alex/meshes/castor_asm_3.dae"/>
     <xacro:property name="castor_mass" value="0.001"/>
     <xacro:property name="castor_height" value="0.025"/>
@@ -150,5 +154,5 @@
     <!-- Pan Mechanism Properties -->
     <xacro:property name="pan_mechanism_mesh_path"
-                    value="package://alex_description/models/pan_asm_2.dae"/>
+                    value="model://alex/meshes/pan_asm_2.dae"/>
     <xacro:property name="pan_mechanism_mass" value="0.005"/>
     <xacro:property name="pan_mechanism_width_x" value="0.016"/>
@@ -175,5 +179,5 @@
     <!-- Tilt Mechanism Properties -->
     <xacro:property name="tilt_mechanism_mesh_path"
-                    value="package://alex_description/models/tilt_asm.dae"/>
+                    value="model://alex/meshes/tilt_asm.dae"/>
     <xacro:property name="tilt_mechanism_mass" value="0.005"/>
     <xacro:property name="tilt_mechanism_width_x" value="0.016"/>
@@ -192,5 +196,5 @@
     <!-- Camera Module Properties -->
     <xacro:property name="camera_module_mesh_path"
-                    value="package://alex_description/models/camera_asm.dae"/>
+                    value="model://alex/meshes/camera_asm.dae"/>
     <xacro:property name="camera_module_mass" value="0.005"/>
     <xacro:property name="camera_module_width_x" value="0.02375"/>
@@ -230,11 +234,4 @@
     <link name="base_link">
         <pose>0 0 ${wheel_radius} 0 0 0</pose>
-        <visual>
-            <origin rpy="0 0 0" xyz="0 0 0"/>
-            <geometry>
-                <box size="0.01 0.01 0.01"/>
-            </geometry>
-            <material name="red"/>
-        </visual>
     </link>
     <link name="chassis">
@@ -359,5 +356,5 @@
     	<child link="right_wheel"/>
     	<xacro:right_wheel_joint_origin/>
-        <limit effort="1.0" velocity="0.45"/>
+        <limit effort="0.1" velocity="0.45"/>
         <xacro:z_axis/>
         <joint_properties damping="1.0" friction="1.0"/>
@@ -388,5 +385,5 @@
     	<child link="left_wheel"/>
     	<xacro:left_wheel_joint_origin/>
-        <limit effort="1.0" velocity="0.45"/>
+        <limit effort="0.1" velocity="0.45"/>
         <xacro:z_axis/>
         <joint_properties damping="1.0" friction="1.0"/>
