Commit message: Add IMU and change web controller to work with sim

File: src/robotics_configurations/alex_description/robots/alex.urdf.xacro (robot description, xacro)
@@ -212,356 +212,8 @@
     </xacro:macro>
     <!-- Camera Sensor Properties -->
-<!--    <xacro:macro name="camera_sensor_joint_origin">-->
-<!--        <origin xyz="0 0.0014 0" rpy="${-pi/2} ${pi} 0"/>-->
-<!--    </xacro:macro>-->
     <xacro:macro name="camera_sensor_joint_origin">
         <origin xyz="0 0.0014 0" rpy="${pi} 0 ${pi/2}"/>
     </xacro:macro>
     <xacro:property name="camera_hfov_rad" value="${108*pi/180}"/>
-    <!-- * * * * * * * * * -->
-    <!-- Generic Macros -->
-    <xacro:macro name="x_axis">
-        <axis xyz="1 0 0" rpy="0 0 0"/>
-    </xacro:macro>
-    <xacro:macro name="y_axis">
-        <axis xyz="0 1 0" rpy="0 0 0"/>
-    </xacro:macro>
-    <xacro:macro name="z_axis">
-        <axis xyz="0 0 1" rpy="0 0 0"/>
-    </xacro:macro>
-    <!-- * * * * * * * * * -->
-    <!-- Model Definitions -->
-    <link name="base_link">
-        <pose>0 0 ${wheel_radius} 0 0 0</pose>
-    </link>
-    <link name="chassis">
-        <inertial>
-            <xacro:chassis_origin/>
-            <mass value="${chassis_mass}"/>
-            <inertia ixx="${chassis_ixx}" ixy="0.0" ixz="0.0" iyy="${chassis_iyy}" iyz="0.0" izz="${chassis_izz}"/>
-        </inertial>
-        <visual>
-            <origin xyz="0 0 0" rpy="0 0 0"/>
-            <geometry>
-<!--                <box size="${chassis_width_x} ${chassis_depth_y} ${chassis_height_z}"/>-->
-                <mesh filename="${chassis_mesh_path}"/>
-            </geometry>
-            <material name="black"/>
-        </visual>
-        <collision>
-            <xacro:chassis_origin/>
-            <geometry>
-                <box size="${chassis_width_x} ${chassis_depth_y} ${chassis_height_z}"/>
-            </geometry>
-        </collision>
-    </link>
-    <joint name="baselink_chassis_joint" type="fixed">
-    	<parent link="base_link"/>
-    	<child link="chassis"/>
-    	<xacro:chassis_joint_origin/>
-	</joint>
-    <gazebo reference="chassis">
-        <kp>10000.0</kp>
-        <kd>10000.0</kd>
-        <mu1>1.0</mu1>
-        <mu2>1.0</mu2>
-    </gazebo>
-    <link name="ep">
-        <inertial>
-            <xacro:ep_box_origin/>
-            <mass value="${ep_mass}"/>
-            <inertia ixx="${ep_ixx}" ixy="0.0" ixz="0.0" iyy="${ep_iyy}" iyz="0.0" izz="${ep_izz}"/>
-        </inertial>
-        <visual>
-            <origin xyz="0 0 0" rpy="0 0 0"/>
-            <geometry>
-<!--                <box size="${ep_width_x} ${ep_depth_y} ${ep_height_z}"/>-->
-                <mesh filename="${ep_mesh_path}"/>
-            </geometry>
-            <material name="black"/>
-        </visual>
-        <collision>
-            <xacro:ep_box_origin/>
-            <geometry>
-                <box size="${ep_width_x} ${ep_depth_y} ${ep_height_z}"/>
-            </geometry>
-        </collision>
-    </link>
-    <joint name="chassis_ep_joint" type="fixed">
-    	<parent link="chassis"/>
-    	<child link="ep"/>
-<!--    	<xacro:ep_joint_origin/>-->
-	</joint>
-    <gazebo reference="ep">
-        <kp>10000.0</kp>
-        <kd>10000.0</kd>
-        <mu1>1.0</mu1>
-        <mu2>1.0</mu2>
-    </gazebo>
-    <link name="pt4">
-        <inertial>
-            <xacro:pt4_box_origin/>
-            <mass value="${pt4_mass}"/>
-            <inertia ixx="${pt4_ixx}" ixy="0.0" ixz="0.0" iyy="${pt4_iyy}" iyz="0.0" izz="${pt4_izz}"/>
-        </inertial>
-        <visual>
-            <origin xyz="0 0 0" rpy="0 0 0"/>
-            <geometry>
-<!--                <box size="${pt4_width_x} ${pt4_depth_y} ${pt4_height_z}"/>-->
-                <mesh filename="${pt4_mesh_path}"/>
-            </geometry>
-            <material name="black"/>
-        </visual>
-        <collision>
-            <xacro:pt4_box_origin/>
-            <geometry>
-                <box size="${pt4_width_x} ${pt4_depth_y} ${pt4_height_z}"/>
-            </geometry>
-        </collision>
-    </link>
-    <joint name="chassis_pt4_joint" type="fixed">
-    	<parent link="chassis"/>
-    	<child link="pt4"/>
-<!--    	<xacro:pt4_joint_origin/>-->
-	</joint>
-    <gazebo reference="pt4">
-        <kp>10000.0</kp>
-        <kd>10000.0</kd>
-        <mu1>1.0</mu1>
-        <mu2>1.0</mu2>
-    </gazebo>
-    <link name="right_wheel">
-        <inertial>
-            <origin rpy="0 0 0" xyz="0 0 0"/>
-            <mass value="${wheel_mass}"/>
-            <inertia ixx="${wheel_ixx}" ixy="0.0" ixz="0.0" iyy="${wheel_iyy}" iyz="0.0" izz="${wheel_izz}"/>
-        </inertial>
-        <visual>
-            <xacro:right_wheel_mesh_origin/>
-            <geometry>
-                <mesh filename="${wheel_mesh_path}"/>
-<!--                <cylinder radius="${wheel_radius}" length="${wheel_width}"/>-->
-            </geometry>
-            <material name="black"/>
-        </visual>
-        <collision>
-            <origin rpy="0 0 0" xyz="0 0 0"/>
-            <geometry>
-                <cylinder radius="${wheel_radius}" length="${wheel_width}"/>
-            </geometry>
-        </collision>
-    </link>
-    <joint name="baselink_right_wheel_joint" type="continuous">
-    	<parent link="base_link"/>
-    	<child link="right_wheel"/>
-    	<xacro:right_wheel_joint_origin/>
-        <limit effort="0.1" velocity="0.45"/>
-        <xacro:z_axis/>
-        <joint_properties damping="1.0" friction="1.0"/>
-	</joint>
-    <link name="left_wheel">
-        <inertial>
-            <origin rpy="0 0 0" xyz="0 0 0"/>
-            <mass value="${wheel_mass}"/>
-            <inertia ixx="${wheel_ixx}" ixy="0.0" ixz="0.0" iyy="${wheel_iyy}" iyz="0.0" izz="${wheel_izz}"/>
-        </inertial>
-        <visual>
-            <xacro:left_wheel_mesh_origin/>
-            <geometry>
-                <mesh filename="${wheel_mesh_path}"/>
-<!--                <cylinder radius="${wheel_radius}" length="${wheel_width}"/>-->
-            </geometry>
-            <material name="black"/>
-        </visual>
-        <collision>
-            <origin rpy="0 0 0" xyz="0 0 0"/>
-            <geometry>
-                <cylinder radius="${wheel_radius}" length="${wheel_width}"/>
-            </geometry>
-        </collision>
-    </link>
-    <joint name="baselink_left_wheel_joint" type="continuous">
-    	<parent link="base_link"/>
-    	<child link="left_wheel"/>
-    	<xacro:left_wheel_joint_origin/>
-        <limit effort="0.1" velocity="0.45"/>
-        <xacro:z_axis/>
-        <joint_properties damping="1.0" friction="1.0"/>
-	</joint>
-    <link name="castor">
-        <inertial>
-            <xacro:castor_collision_origin/>
-            <mass value="${castor_mass}"/>
-            <inertia ixx="${castor_ixx}" ixy="0.0" ixz="0.0" iyy="${castor_iyy}" iyz="0.0" izz="${castor_izz}"/>
-        </inertial>
-        <visual>
-            <xacro:castor_mesh_origin/>
-            <geometry>
-                <mesh filename="${castor_mesh_path}"/>
-            </geometry>
-        </visual>
-        <collision>
-            <xacro:castor_collision_origin/>
-            <geometry>
-                <cylinder radius="${castor_radius}" length="${castor_height}"/>
-            </geometry>
-        </collision>
-    </link>
-    <joint name="baselink_castor_joint" type="continuous">
-    	<parent link="base_link"/>
-    	<child link="castor"/>
-    	<xacro:castor_joint_origin/>
-        <limit effort="1.0" velocity="0.45"/>
-        <xacro:z_axis/>
-        <joint_properties damping="1.0" friction="1.0"/>
-	</joint>
-    <gazebo reference="castor">
-        <kp>10000.0</kp>
-        <kd>10000.0</kd>
-        <mu1>10.0</mu1>
-        <mu2>10.0</mu2>
-    </gazebo>
-    <link name="castor_wheel">
-        <inertial>
-            <origin rpy="0 0 0" xyz="0 0 0"/>
-            <mass value="${castor_wheel_mass}"/>
-            <inertia ixx="${castor_wheel_ixx}" ixy="0.0" ixz="0.0" iyy="${castor_wheel_iyy}" iyz="0.0" izz="${castor_wheel_izz}"/>
-        </inertial>
-        <collision>
-            <origin rpy="0 0 0" xyz="0 0 0"/>
-            <geometry>
-                <cylinder radius="${castor_wheel_radius}" length="${castor_wheel_width}"/>
-            </geometry>
-        </collision>
-    </link>
-    <joint name="castor_castorwheel_joint" type="continuous">
-    	<parent link="castor"/>
-    	<child link="castor_wheel"/>
-    	<xacro:castor_wheel_joint_origin/>
-        <limit effort="1.0" velocity="0.45"/>
-        <xacro:z_axis/>
-        <joint_properties damping="1.0" friction="1.0"/>
-	</joint>
-    <link name="pan_mechanism">
-        <inertial>
-            <xacro:pan_mechanism_origin/>
-            <mass value="${pan_mechanism_mass}"/>
-            <inertia ixx="${pan_mechanism_ixx}" ixy="0.0" ixz="0.0" iyy="${pan_mechanism_iyy}" iyz="0.0" izz="${pan_mechanism_izz}"/>
-        </inertial>
-        <visual>
-<!--            <xacro:pan_mechanism_origin/>-->
-            <origin rpy="0 0 0" xyz="0 0 0"/>
-            <geometry>
-<!--                <box size="${pan_mechanism_width_x} ${pan_mechanism_depth_y} ${pan_mechanism_height_z}"/>-->
-                <mesh filename="${pan_mechanism_mesh_path}"/>
-            </geometry>
-            <material name="black"/>
-        </visual>
-        <collision>
-            <xacro:pan_mechanism_origin/>
-            <geometry>
-                <box size="${pan_mechanism_width_x} ${pan_mechanism_depth_y} ${pan_mechanism_height_z}"/>
-            </geometry>
-        </collision>
-    </link>
-    <joint name="pan_mechanism_joint" type="revolute">
-    	<parent link="chassis"/>
-    	<child link="pan_mechanism"/>
-    	<xacro:pan_mechanism_joint_origin/>
-        <limit lower="${-pi/2}" upper="${pi/2}" effort="1.0" velocity="${100*pi/180}"/>
-        <xacro:y_axis/>
-        <joint_properties damping="1.0" friction="1.0"/>
-	</joint>
-    <link name="tilt_mechanism">
-        <inertial>
-            <xacro:tilt_mechanism_origin/>
-            <mass value="${tilt_mechanism_mass}"/>
-            <inertia ixx="${tilt_mechanism_ixx}" ixy="0.0" ixz="0.0" iyy="${tilt_mechanism_iyy}" iyz="0.0" izz="${tilt_mechanism_izz}"/>
-        </inertial>
-        <visual>
-<!--            <xacro:tilt_mechanism_origin/>-->
-            <origin rpy="0 0 0" xyz="0 0 0"/>
-            <geometry>
-<!--                <box size="${tilt_mechanism_width_x} ${tilt_mechanism_depth_y} ${tilt_mechanism_height_z}"/>-->
-                <mesh filename="${tilt_mechanism_mesh_path}"/>
-            </geometry>
-            <material name="black"/>
-        </visual>
-        <collision>
-            <xacro:tilt_mechanism_origin/>
-            <geometry>
-                <box size="${tilt_mechanism_width_x} ${tilt_mechanism_depth_y} ${tilt_mechanism_height_z}"/>
-            </geometry>
-        </collision>
-    </link>
-    <joint name="tilt_mechanism_joint" type="revolute">
-    	<parent link="pan_mechanism"/>
-    	<child link="tilt_mechanism"/>
-    	<xacro:tilt_mechanism_joint_origin/>
-        <limit lower="${-pi/2}" upper="${pi/2}" effort="1.0" velocity="${100*pi/180}"/>
-        <xacro:y_axis/>
-        <joint_properties damping="1.0" friction="1.0"/>
-	</joint>
-    <xacro:gazebo_wheel_params link_ref="left_wheel"/>
-    <xacro:gazebo_wheel_params link_ref="right_wheel"/>
-    <xacro:gazebo_castor_wheel_params link_ref="castor_wheel"/>
-    <xacro:servo_params link_ref="pan_mechanism"/>
-    <xacro:servo_params link_ref="tilt_mechanism"/>
-    <xacro:macro name="servo_transmission_macro" params="joint servo_type">
-        <transmission name="${servo_type}_transmission">
-            <type>transmission_interface/SimpleTransmission</type>
-            <joint name="${joint}">
-                <hardwareInterface>hardware_interface/PositionJointInterface</hardwareInterface>
-            </joint>
-            <actuator name="${servo_type}_servo_actuator">
-                <hardwareInterface>hardware_interface/PositionJointInterface</hardwareInterface>
-                <mechanicalReduction>1</mechanicalReduction>
-            </actuator>
-        </transmission>
-    </xacro:macro>
-    <xacro:servo_transmission_macro joint="pan_mechanism_joint" servo_type="pan" />
-    <xacro:servo_transmission_macro joint="tilt_mechanism_joint" servo_type="tilt" />
-    <link name="camera_module">
-        <inertial>
-            <xacro:camera_module_box_origin/>
-            <mass value="${camera_module_mass}"/>
-            <inertia ixx="${camera_module_ixx}" ixy="0.0" ixz="0.0" iyy="${camera_module_iyy}" iyz="0.0" izz="${camera_module_izz}"/>
-        </inertial>
-        <visual>
-<!--            <xacro:camera_module_box_origin/>-->
-            <origin rpy="0 0 0" xyz="0 0 0"/>
-            <geometry>
-<!--                <box size="${camera_module_width_x} ${camera_module_depth_y} ${camera_module_height_z}"/>-->
-                <mesh filename="${camera_module_mesh_path}"/>
-            </geometry>
-            <material name="black"/>
-        </visual>
-        <collision>
-            <xacro:camera_module_box_origin/>
-            <geometry>
-                <box size="${camera_module_width_x} ${camera_module_depth_y} ${camera_module_height_z}"/>
-            </geometry>
-        </collision>
-    </link>
-    <joint name="camera_module_joint" type="fixed">
-    	<parent link="tilt_mechanism"/>
-    	<child link="camera_module"/>
-    	<xacro:camera_module_joint_origin/>
-	</joint>
-    <link name="camera_sensor">
-        <visual>
-            <origin rpy="0 0 0" xyz="0 0 0"/>
-            <geometry>
-                <box size="0.001 0.001 0.001"/>
-            </geometry>
-            <material name="red"/>
-        </visual>
-    </link>
-    <joint name="camera_sensor_joint" type="fixed">
-    	<parent link="camera_module"/>
-    	<child link="camera_sensor"/>
-    	<xacro:camera_sensor_joint_origin/>
-	</joint>
-    <!-- camera -->
     <gazebo reference="camera_sensor">
         <sensor type="camera" name="camera1">
@@ -587,5 +239,5 @@
                 </noise>
             </camera>
-            <plugin name="camera_controller" filename="libgazebo_ros_camera.so">
+            <plugin filename="libgazebo_ros_camera.so" name="camera_controller">
                 <alwaysOn>true</alwaysOn>
                 <updateRate>0.0</updateRate>
@@ -603,3 +255,384 @@
         </sensor>
     </gazebo>
+<!--    <xacro:macro name="camera_sensor_joint_origin">-->
+<!--        <origin xyz="0 0.0014 0" rpy="${-pi/2} ${pi} 0"/>-->
+<!--    </xacro:macro>-->
+    <!-- * * * * * * * * * -->
+    <!-- Generic Macros -->
+    <xacro:macro name="x_axis">
+        <axis xyz="1 0 0" rpy="0 0 0"/>
+    </xacro:macro>
+    <xacro:macro name="y_axis">
+        <axis xyz="0 1 0" rpy="0 0 0"/>
+    </xacro:macro>
+    <xacro:macro name="z_axis">
+        <axis xyz="0 0 1" rpy="0 0 0"/>
+    </xacro:macro>
+    <!-- * * * * * * * * * -->
+    <!-- Model Definitions -->
+    <link name="base_link">
+        <pose>0 0 ${wheel_radius} 0 0 0</pose>
+    </link>
+    <link name="chassis">
+        <inertial>
+            <xacro:chassis_origin/>
+            <mass value="${chassis_mass}"/>
+            <inertia ixx="${chassis_ixx}" ixy="0.0" ixz="0.0" iyy="${chassis_iyy}" iyz="0.0" izz="${chassis_izz}"/>
+        </inertial>
+        <visual>
+            <origin xyz="0 0 0" rpy="0 0 0"/>
+            <geometry>
+<!--                <box size="${chassis_width_x} ${chassis_depth_y} ${chassis_height_z}"/>-->
+                <mesh filename="${chassis_mesh_path}"/>
+            </geometry>
+            <material name="black"/>
+        </visual>
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