Commit message: Add new daes, fix model directories

File: src/robotics_configurations/alex_description/robots/alex.urdf (robot description, URDF)
Before this commit: robot alex, 12 links, 11 joints
Links:
- added link imu_link; visual box size=0.001 0.001 0.001
- link camera_module: geometry collision box size=0.02375 0.0124 0.02375; visual mesh filename=model://alex/meshes/camera_asm_2_dessimate.dae
- link castor: geometry collision cylinder length=0.025 radius=0.0162; visual mesh filename=model://alex/meshes/castor_asm_3_dessimate.dae
- link chassis: geometry collision box size=0.192 0.059 0.276; visual mesh filename=model://alex/meshes/chassis_asm_dessimate.dae
- link ep: geometry collision box size=0.1015 0.018 0.134; visual box size=0.1015 0.018 0.134
- link left_wheel: geometry collision cylinder length=0.029 radius=0.0375; visual mesh filename=model://alex/meshes/wheel_asm_decimate_3.dae
- link pan_mechanism: geometry collision box size=0.016 0.0385 0.048; visual mesh filename=model://alex/meshes/pan_asm_2_dessimate_2.dae
- link pt4: geometry collision box size=0.0995 0.034 0.132; visual box size=0.0995 0.034 0.132
- link right_wheel: geometry collision cylinder length=0.029 radius=0.0375; visual mesh filename=model://alex/meshes/wheel_asm_decimate_3.dae
- link tilt_mechanism: geometry collision box size=0.016 0.0385 0.048; visual mesh filename=model://alex/meshes/tilt_asm_dessimate.dae
Joints:
- added joint ep_imu_joint: type fixed, parent ep, child imu_link, origin xyz=0 -0.0085 0 rpy=0 0 0

File: src/robotics_configurations/alex_description/robots/alex.urdf.xacro (robot description, xacro)
@@ -35,5 +35,5 @@
     <!-- Chassis Properties -->
     <xacro:property name="chassis_mesh_path"
-                    value="model://alex/meshes/chassis_asm.dae"/>
+                    value="model://alex/meshes/chassis_asm_dessimate.dae"/>
     <xacro:property name="chassis_mass" value="0.650"/>
     <xacro:property name="chassis_width_x" value="0.192"/>
@@ -48,10 +48,10 @@
     </xacro:macro>
     <xacro:macro name="chassis_joint_origin">
-        <origin xyz="-0.068 0 0.056475" rpy="${pi/2} 0 ${-pi/2}"/>
+        <origin xyz="-0.068 0 0.056475" rpy="${pi/2} 0 ${-pi/2}"/>\
     </xacro:macro>
     <!-- * * * * * * * * * -->
     <!-- Expansion Plate Properties -->
     <xacro:property name="ep_mesh_path"
-                    value="model://alex/meshes/EP_asm.dae"/>
+                    value="model://alex/meshes/EP_asm_decimate_4.dae"/>
     <xacro:property name="ep_mass" value="0.05"/>
     <xacro:property name="ep_width_x" value="0.1015"/>
@@ -68,5 +68,5 @@
     <!-- pi-top [4] Properties -->
     <xacro:property name="pt4_mesh_path"
-                    value="model://alex/meshes/4_asm_2.dae"/>
+                    value="model://alex/meshes/4_asm_2_dessimate.dae"/>
     <xacro:property name="pt4_mass" value="0.390"/>
     <xacro:property name="pt4_width_x" value="0.0995"/>
@@ -82,5 +82,5 @@
     <!-- Wheel Properties -->
     <xacro:property name="wheel_mesh_path"
-                    value="model://alex/meshes/wheel_asm.dae"/>
+                    value="model://alex/meshes/wheel_asm_decimate_3.dae"/>
     <xacro:property name="wheel_mass" value="0.01"/>
     <xacro:property name="wheel_width" value="0.029"/>
@@ -116,5 +116,5 @@
     <!-- Castor Properties -->
     <xacro:property name="castor_mesh_path"
-                    value="model://alex/meshes/castor_asm_3.dae"/>
+                    value="model://alex/meshes/castor_asm_3_dessimate.dae"/>
     <xacro:property name="castor_mass" value="0.001"/>
     <xacro:property name="castor_height" value="0.025"/>
@@ -154,5 +154,5 @@
     <!-- Pan Mechanism Properties -->
     <xacro:property name="pan_mechanism_mesh_path"
-                    value="model://alex/meshes/pan_asm_2.dae"/>
+                    value="model://alex/meshes/pan_asm_2_dessimate_2.dae"/>
     <xacro:property name="pan_mechanism_mass" value="0.005"/>
     <xacro:property name="pan_mechanism_width_x" value="0.016"/>
@@ -179,5 +179,5 @@
     <!-- Tilt Mechanism Properties -->
     <xacro:property name="tilt_mechanism_mesh_path"
-                    value="model://alex/meshes/tilt_asm.dae"/>
+                    value="model://alex/meshes/tilt_asm_dessimate.dae"/>
     <xacro:property name="tilt_mechanism_mass" value="0.005"/>
     <xacro:property name="tilt_mechanism_width_x" value="0.016"/>
@@ -196,5 +196,5 @@
     <!-- Camera Module Properties -->
     <xacro:property name="camera_module_mesh_path"
-                    value="model://alex/meshes/camera_asm.dae"/>
+                    value="model://alex/meshes/camera_asm_2_dessimate.dae"/>
     <xacro:property name="camera_module_mass" value="0.005"/>
     <xacro:property name="camera_module_width_x" value="0.02375"/>
@@ -315,6 +315,6 @@
             <origin xyz="0 0 0" rpy="0 0 0"/>
             <geometry>
-                <box size="${ep_width_x} ${ep_depth_y} ${ep_height_z}"/>
-<!--                <mesh filename="${ep_mesh_path}"/>-->
+<!--                <box size="${ep_width_x} ${ep_depth_y} ${ep_height_z}"/>-->
+                <mesh filename="${ep_mesh_path}"/>
             </geometry>
             <material name="black"/>
@@ -347,6 +347,6 @@
             <origin xyz="0 0 0" rpy="0 0 0"/>
             <geometry>
-                <box size="${pt4_width_x} ${pt4_depth_y} ${pt4_height_z}"/>
-<!--                <mesh filename="${pt4_mesh_path}"/>-->
+<!--                <box size="${pt4_width_x} ${pt4_depth_y} ${pt4_height_z}"/>-->
+                <mesh filename="${pt4_mesh_path}"/>
             </geometry>
             <material name="black"/>
